File: INA2xx_Breakout-Board.kicad_pcb (KiCad board)
At the start: 2 copper layers, 20.3 x 15.2 mm, 3 parts, among them J1 Conn_01x05_Male, J2 Conn_01x05_Male, U1 INA226

Commit message: Mod: Bottom filled zone, added my logo to the solder mask and exported v-cuts
Parts:
- added G***: LOGO, drawings:elektronik-emblem_3x3.5_solder, B.Cu at (152.4, 97.2)
Routing:
- added copper zone on B.Cu, net (none)

Commit message: Add: Project name and revision on the bottom solder mask, modified .gitignore
Other:
- board text added: "Prj: ${TITLE} Rev: ${REVISION}"
Changed lines of the file:
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@@
     (effects (font (size 1.5 1.5) (thickness 0.3)))
+  )
+  (gr_text "Prj: ${TITLE}\nRev: ${REVISION}" (at 152.4 105.41) (layer "B.Mask")
+    (effects (font (size 0.4 0.4) (thickness 0.1)) (justify mirror))
   )
   (segment (start 144.78 96.52) (end 148.86 100.6) (width 0.25) (layer "F.Cu") (net 1))
